File: rocket2-afs.kicad_pcb (KiCad board)
At the start: 4 copper layers, 70 x 50 mm, 72 parts, among them J1 ARMING_PLUG, J2 POWER, J3 E-MATCH_DROGUE, J4 SWD, J5 E-MATCH_RECOVERY, Q1 Q_NMOS_GSD, Q2 Q_NMOS_GSD, Q3 Q_NMOS_GSD, Q4 Q_NMOS_GSD, Q5 Q_NMOS_GSD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

Commit message: Changed Debug Symbol to UCIRP-L Library footrpint
Connections:
- J4 pad 4: DEBUCK_SWCLK -> DEBUG_SWCLK

Commit message: Final tweaks
Connections:
- U1 pad 49: DEBUCK_SWCLK -> DEBUG_SWCLK
Routing:
- net DEBUG_SWCLK: track 0.00 -> 31.0 mm, vias 0 -> 1
- net DEBUCK_SWCLK: track 31.0 -> 0.00 mm, vias 1 -> 0
Other:
- board text added: "UCI Rocket Project - Avionics Avionics Flight Sensors v2.1 03/12/2024"
- board text removed: "UCI Rocket Project - Avionics Avionics Flight System Betelgeuse v2.1 03/12/2024"

Commit message: Added GPS RESET pullup resistor to PCB
Parts:
- added R23: 10k, Resistor_SMD:R_0603_1608Metric, F.Cu at (165.6, 87.3)
Routing:
- net +3.3V: track 73.2 -> 76.3 mm
- net GPS_RESET: track 23.8 -> 25.7 mm
